Commit message: Integrated sensors and updated robot model

File: install/aqua_robot_gazebo/share/aqua_robot_gazebo/urdf/aqua_robot.urdf (robot description, URDF)
Before this commit: robot aqua_waste_robot, 6 links, 5 joints
Links:
- added link gps_link, mass 0.05
- added link imu_link, mass 0.05
- added link lidar_link, mass 0.2; collision cylinder length=0.05 radius=0.05; visual cylinder length=0.05 radius=0.05
Joints:
- added joint gps_joint: type fixed, parent base_link, child gps_link, origin xyz=0 0 0.08 rpy=0 0 0
- added joint imu_joint: type fixed, parent base_link, child imu_link, origin xyz=0 0 0.05 rpy=0 0 0
- added joint lidar_joint: type fixed, parent mast, child lidar_link, origin xyz=0 0 0.25 rpy=0 0 0

Commit message: clean repo structure - removed build install log

File: install/aqua_robot_gazebo/share/aqua_robot_gazebo/urdf/aqua_robot.urdf (robot description, URDF)
Before this commit: robot aqua_waste_robot, 9 links, 8 joints
Links:
- link mast: geometry collision cylinder length=0.45 radius=0.025; visual cylinder length=0.45 radius=0.025
