Commit message: Update aqua_robot_multi.urdf.xacro

File: src/aqua_robot_gazebo/urdf/aqua_robot_multi.urdf.xacro (robot description, xacro)
@@ -1,4 +1,5 @@
 <?xml version="1.0"?>
 <robot name="aqua_waste_robot" xmlns:xacro="http://www.ros.org/wiki/xacro">
+<xacro:arg name="robot_ns" default="aqua_robot"/>
   <!-- ============================================================ -->
   <!--  MATERIALS                                                    -->
@@ -24,4 +25,7 @@
   <material name="dark_prop">
     <color rgba="0.2 0.2 0.2 1"/>
+  </material>
+  <material name="green">
+    <color rgba="0.0 1.0 0.0 1.0"/>
   </material>
   <!-- ============================================================ -->
@@ -36,10 +40,10 @@
     <visual>
       <origin xyz="0 0 0" rpy="0 0 0"/>
-      <geometry><box size="0.9 0.5 0.22"/></geometry>
+      <geometry><box size="0.9 0.5 0.05"/></geometry>
       <material name="blue_body"/>
     </visual>
     <collision>
       <origin xyz="0 0 0" rpy="0 0 0"/>
-      <geometry><box size="0.9 0.5 0.22"/></geometry>
+      <geometry><box size="0.9 0.5 0.05"/></geometry>
     </collision>
   </link>
@@ -103,5 +107,5 @@
     <origin xyz="0 0 0" rpy="0 0 0"/>
     <geometry>
-      <cylinder radius="0.025" length="0.45"/>
+      <cylinder radius="0.025" length="0.28"/>
     </geometry>
     <material name="grey_frame"/>
@@ -109,5 +113,5 @@
   <collision>
     <geometry>
-      <cylinder radius="0.025" length="0.45"/>
+      <cylinder radius="0.025" length="0.28"/>
     </geometry>
   </collision>
@@ -116,5 +120,5 @@
     <parent link="base_link"/>
     <child link="mast"/>
-    <origin xyz="0.1 0 0.30" rpy="0 0 0"/>
+    <origin xyz="0.1 0 0.07" rpy="0 0 0"/>
   </joint>
   <!-- ============================================================ -->
@@ -135,5 +139,5 @@
     <parent link="mast"/>
     <child link="camera_link"/>
-    <origin xyz="0 0 0.25" rpy="0 0 0"/>
+    <origin xyz="0 0 0.20" rpy="0 0 0"/>
   </joint>
   <!-- ============================================================ -->
@@ -147,19 +151,25 @@
                izz="0.001"/>
     </inertial>
-    <visual>
-      <geometry>
-        <cylinder radius="0.05" length="0.05"/>
-      </geometry>
-    </visual>
-    <collision>
-      <geometry>
-        <cylinder radius="0.05" length="0.05"/>
-      </geometry>
-    </collision>
+<visual>
+  <geometry>
+    <cylinder radius="0.05" length="0.05"/>
+  </geometry>
+  <material>
+    <ambient>0 1 0 1</ambient>
+    <diffuse>0 1 0 1</diffuse>
+    <specular>0.1 0.1 0.1 1</specular>
+    <emissive>0 0.3 0 1</emissive>
+  </material>
+</visual>
+<collision>
+  <geometry>
+    <cylinder radius="0.05" length="0.05"/>
+  </geometry>
+</collision>
   </link>
   <joint name="lidar_joint" type="fixed">
     <parent link="mast"/>
     <child link="lidar_link"/>
-    <origin xyz="0 0 0.25" rpy="0 0 0"/>
+    <origin xyz="0 0 0.15" rpy="0 0 0"/>
   </joint>
   <!-- IMU -->
@@ -195,20 +205,21 @@
   <!-- ============================================================ -->
   <gazebo reference="lidar_link">
-    <sensor type="ray" name="lidar_sensor">
-      <update_rate>10</update_rate>
+    <material>Gazebo/Green</material>
+   <sensor type="ray" name="lidar_sensor">
+  <update_rate>10</update_rate>
 <ray>
   <scan>
-    <horizontal>
-      <samples>360</samples>
-      <resolution>1</resolution>
-      <min_angle>-3.14159</min_angle>
-      <max_angle>3.14159</max_angle>
-    </horizontal>
-    <vertical>
-      <samples>1</samples>
-      <resolution>1</resolution>
-      <min_angle>0.0</min_angle>
-      <max_angle>0.0</max_angle>
-    </vertical>
+<horizontal>
+  <samples>360</samples>
+  <resolution>1</resolution>
+  <min_angle>-3.14159</min_angle>
+  <max_angle>3.14159</max_angle>
+</horizontal>
+<vertical>
+  <samples>1</samples>
+  <resolution>1</resolution>
+  <min_angle>0.0</min_angle>
+  <max_angle>0.0</max_angle>
+</vertical>
   </scan>
   <range>
@@ -221,9 +232,7 @@
         filename="libgazebo_ros_ray_sensor.so">
   <ros>
-    <namespace>/aqua_robot</namespace>
+    <namespace>$(arg robot_ns)</namespace>
   </ros>
-  <output_type>sensor_msgs/LaserScan</output_type>
-  <topic_name>scan</topic_name>
-  <frame_name>lidar_link</frame_name>
+<output_type>sensor_msgs/LaserScan</output_type><topic_name>scan</topic_name><frame_name>lidar_link</frame_name>
 </plugin>
     </sensor>
@@ -233,13 +242,13 @@
       <always_on>true</always_on>
       <update_rate>50</update_rate>
-      <plugin name="imu_plugin"
-              filename="libgazebo_ros_imu_sensor.so">
-        <ros>
-          <namespace>/aqua_robot</namespace>
-        </ros>
-        <topic_name>imu</topic_name>
-        <frame_name>imu_link</frame_name>
-      </plugin>
-    </sensor>
+  <plugin name="imu_plugin"
+          filename="libgazebo_ros_imu_sensor.so">
+    <ros>
+      <namespace>$(arg robot_ns)</namespace>
+    </ros>
+    <topic_name>imu</topic_name>
+    <frame_name>imu_link</frame_name>
+  </plugin>
+</sensor>
   </gazebo>
 <gazebo reference="gps_link">
@@ -247,11 +256,11 @@
     <always_on>true</always_on>
     <update_rate>5</update_rate>
-    <plugin name="gps_plugin"
-            filename="libgazebo_ros_gps_sensor.so">
-      <ros>
-        <namespace>/aqua_robot</namespace>
-      </ros>
-      <frame_name>gps_link</frame_name>
-    </plugin>
+<plugin name="gps_plugin"
+        filename="libgazebo_ros_gps_sensor.so">
+  <ros>
+      <namespace>$(arg robot_ns)</namespace>
+  </ros>
+  <frame_name>gps_link</frame_name>
+</plugin>
   </sensor>
 </gazebo>
@@ -338,14 +347,14 @@
 <gazebo>
   <plugin name="planar_move" filename="libgazebo_ros_planar_move.so">
-    <ros>
-      <namespace>/aqua_robot</namespace>
-    </ros>
-    <update_rate>30</update_rate>
-    <publish_odom>true</publish_odom>
-    <publish_odom_tf>true</publish_odom_tf>
-    <command_topic>cmd_vel</command_topic>
-    <odometry_topic>odom</odometry_topic>
-    <odometry_frame>odom</odometry_frame>
-    <robot_base_frame>base_link</robot_base_frame>
+<ros>
+   <namespace>$(arg robot_ns)</namespace>
+</ros>
+<update_rate>30</update_rate>
+<publish_odom>true</publish_odom>
+<publish_odom_tf>true</publish_odom_tf>
+<command_topic>cmd_vel</command_topic>
+<odometry_topic>odom</odometry_topic>
+<odometry_frame>odom</odometry_frame>
+<robot_base_frame>base_link</robot_base_frame>
   </plugin>
 </gazebo>
